File: Aqua BMS Monitor (2).kicad_sch (KiCad schematic)
At the start: 206 parts, among them J4 Conn_01x04, J5 Conn_01x04, Q1 NMOS, Q10 NMOS, Q11 NMOS, Q13 NMOS, Q14 NMOS, Q2 PMOS, Q3 PMOS, Q4 NMOS, Q5 NMOS, Q6 NPN, Q7 NMOS, Q8 PMOS, Q9 NMOS, SW1 Button, SW1 SW_Push, SW2 SW_Push, U1 BQ76952PFBR, U2 STM32F205RETx

Commit message: Updated June 17
Parts:
- removed D19: 5V, symbol Device:D_Zener
- added C41, C42, C44: 0.1 uF, symbol Device:C
- added C43: 470 pF, symbol Device:C
- added D18: 10 V, symbol Device:D_Zener
- added F1: Fuse, symbol Device:Fuse
- added Q12: NMOS, symbol Simulation_SPICE:NMOS
- added R55: 5.1k, symbol Device:R
- added R56: 100k, symbol Device:R
- added TH5: Thermistor_US, symbol Device:Thermistor_US
- added TP17, TP19: TestPoint, symbol Connector:TestPoint
Connections:
- net BAT + is gone; now on net PACK +: R49.2
- net VSS is gone; now on net PGND: BQ296115DSGR1.6 (VSS), BQ296115DSGR1.9 (PWPD), BQ296115DSGR2.6 (VSS), BQ296115DSGR2.9 (PWPD), C00.2, C1-0.2, C1.2, C1.2, C10.2, C11.1, C11.2, C12.2, C13.2, C14.2, C15.2, C16.1, C16.2, C17.2, C17.2, C18.2, C19.2, C2.1, C2.2, C20.2, C21.2, C3.2, C3.2, C33.2, C34.2, C35.1, C36.1, C4.2, C40.2, C5.2, C6.2, C7.2, C7.2, C8.1, C8.2, C9.2, C9.2, Cellin1.1 (Pin_1), J.A1 (GND), J.A12 (GND), J.B1 (GND), J.B12 (GND), J.SH (SHIELD), MainBattIn.2 (Pin_2), MainBattIn1.2 (Pin_2), Q5.3 (S), R15.2, R20.2, R22.1, R4.2, R46.1, R5.2, R5.2, R50.2, R51.1, R52.1, R53.1, R6.2, R7.2, R9.2, RC0.1, RShunt.1, SW1.1, TH3.2, TH4.2, TP6.1, U1.17 (VSS), U2.12 (VSSA), U2.18 (VSS), U2.63 (VSS)
- net FUSE: now also R55.1; no longer R54.1
- net PGND: now also C41.2, C42.2, C43.2, C44.2, D18.2 (A), Q12.3 (S), R56.1, TH5.2
- net SRN: now also C42.1
- net SRP: now also C41.1
- new net: C44.1, D18.1 (K), Q12.2 (G), R54.1, R55.2, R56.2, TP19.1
- new net: F1.1, Q12.1 (D)
- new net HDQ: C43.1, TH5.1, TP17.1
Other:
- note added: "1 uF? ^"
- note added: "100 nF? ->"
- note added: "10k resistor typically connected between PACK+ and LD"
- note added: "ALERT, CFETOFF, DFETOFF, TS1, TS2, TS3, HDQ, DCHG, and DDSG are also for thermistor temp measurement"
- note added: "Backfeeding protection ->"
- note added: "Pre-charge and pre-discharge circuits"
- note added: "Voltage on REGIN should not exceed BAT"
- note added: "Where did you come from -> Overvoltage protection"
- moved on the sheet: BQ296115DSGR2, C35, C36, C37, C38, C39, C40, R48, R49, R50, R51, R52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

Commit message: Updated June 19
Parts:
- added R57, R58: 4.7k, symbol Device:R
- R17: value 0 -> 51
- R56: value 100k -> 20k
Connections:
- net MCU: now also R57.1, R58.1
- net PGND: no longer BQ296115DSGR2.9 (PWPD)
Other:
- note added: "1 uF in datasheet?"
- note added: "<- 150 in datasheet"
- note added: "Why? Reduce power loss through Rds?"
- note removed: "Where did you come from -> Overvoltage protection"
- moved on the sheet: BQ296115DSGR2, C35, C36, C37, C38, C39, C40, C44, D18, F1, Q12, R48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
