File: Aqua BMS Monitor(MAIN).kicad_sch (KiCad schematic)
At the start: 224 parts, among them J1 Conn_01x03, J4 USB_C_Receptacle_USB2.0_14P, J5 SWD_01x04_Pin, Q13 NMOS, Q6 NPN, SW2 SW_Push, SW3 SW_Push, SW4 SW_Push, SW5 SW_Push, SW6 SW_Push, SW7 SW_Push, U1 BQ7695202, U2 STM32F205RETx, U3 AMS1117-3.3, U4 LM66100DCKR, U5 LM66100DCKR, U6 LM66100DCKR, X1 X322516MRB4SI

Commit message: Several changes
- Renamed components in discharge circuit
- Removed blocking fets
- Added physical E-stop switch mechanism
- Added ideal diode and test points
- Renamed components for MCU
- Added final test points
Parts:
- removed DBlokFet1, DBlokFet2: NMOS, easyeda2kicad:NMOS, symbol Simulation_SPICE:NMOS
- removed R63, R64: 51, easyeda2kicad:51_R1206, symbol BQ76952PFBR:R
- added DC3: 47nF, easyeda2kicad:0.1uF_C1210, symbol Device:C
- added DD3: 16V, easyeda2kicad:16V_Zener, symbol Device:D_Zener
- added DFet3: NMOS, easyeda2kicad:NMOS, symbol Simulation_SPICE:NMOS
- added DR4: 10M, easyeda2kicad:10M_R1210, symbol BQ76952PFBR:R
- added DR5: 1k, easyeda2kicad:5.1k_R1210, symbol BQ76952PFBR:R
- added DTVS30, DTVS70: D_TVS_Filled, symbol Device:D_TVS_Filled
- added S1: MHPS2285N, MHPS2285N, symbol MHPS2285N:MHPS2285N
- added TP23: RXTP, symbol Connector:TestPoint
- added TP24: MCUSDATP, symbol Connector:TestPoint
- added TP25: MCUSCLTP, symbol Connector:TestPoint
- added TP56: IDTVSTP, symbol Connector:TestPoint
- added TP57: IDGTP, symbol Connector:TestPoint
- added TP58: IDVSSTP, symbol Connector:TestPoint
- added TP59: VSWDTP, symbol Connector:TestPoint
- added TP60: V_REGUSB, symbol Connector:TestPoint
- added TP61: Vcap1TP, symbol Connector:TestPoint
- added TP62: Vcap2TP, symbol Connector:TestPoint
- added TP63: ALERTTP, symbol Connector:TestPoint
- added TP64: BOOT0TP, symbol Connector:TestPoint
- added TP65: NRSTTP, symbol Connector:TestPoint
- added TP66: MCfetOffTP, symbol Connector:TestPoint
- added TP67: CfetOffTP, symbol Connector:TestPoint
- added TP68: MDfetOffTP, symbol Connector:TestPoint
- added TP69: DfetOffTP, symbol Connector:TestPoint
- added TP70: DCHGTP, symbol Connector:TestPoint
- added TP71: DDSGTP, symbol Connector:TestPoint
- added TP72: RST_SHUTTP, symbol Connector:TestPoint
- added U7: LTC4359-DCB, Package_DFN_QFN:DFN-6-1EP_3x2mm_P0.5mm_EP1.65x1.35mm, symbol Power_Management:LTC4359-DCB
- J1: value Conn_01x03 -> UART Jpins
- TP5: value TestPoint -> TXTP
- renumbered C7 to BC1, C11 to BC2, C12 to BC3, D1 to BD1, D2 to BD2, C27 to BMSC1, SW3 to BOOTSW1, R6 to BR1, C34 to DC1, C35 to DC2, D14 to DD1, D13 to DD2, R43 to DR1, R44 to DR2, R42 to DR3, R41 to DRgate2, R32 to FUSER2, R35 to LDR, D7 to LED1, D10 to LED2, D11 to LED3, D5 to LED4, D6 to LED5, R38 to LEDR1, R65 to LEDR2, R66 to LEDR3, R36 to LEDR4, R37 to LEDR5, C41 to MCUC1, C53 to MCUC10, C58 to MCUC11, C59 to MCUC12, C60 to MCUC13, C61 to MCUC14, C62 to MCUC15, C64 to MCUC16, C63 to MCUC17, C65 to MCUC18, C39 to MCUC19, C42 to MCUC2, C38 to MCUC20, C40 to MCUC21, C43 to MCUC3, C45 to MCUC4, C46 to MCUC5, C47 to MCUC6, C49 to MCUC7, C51 to MCUC8, C52 to MCUC9, R13 to MCUR1, R49 to MCUR2, R48 to MCUR3, R12 to MCUR4, R55 to MCUR5, R56 to MCUR6, D12 to MCUTVS1, D16 to MCUTVS2, SW2 to NRSTSW2, C13 to OSCC1, C15 to OSCC2, C24 to RC1, C20 to RC2, C18 to RC3, C19 to RC4, D8 to RD1, D9 to RD2, R23 to RR1, R22 to RR2, SW4 to SWShunt1, SW5 to SWShunt2, SW6 to SWShunt3, SW7 to SWShunt4, C16 to USBC1, C22 to USBC2, R4 to USBR1, R10 to USBR2, R11 to USBR3
Connections:
- net PGND is gone; now on net VSS: D15.2 (A)
- net ALERT: now also TP63.1
- net CFETOFF: now also S1.6 (COM_2), TP67.1; no longer U2.10 (PC2)
- net DCHG: now also TP70.1
- net DDSG: now also TP71.1
- net DFETOFF: now also S1.3 (COM_1), TP69.1; no longer U2.9 (PC1)
- net DPACK+: now also DC3.1, DFet3.1 (D), U7.1 (OUT)
- net RST_SHUT: now also TP72.1
- net USART1_RX: now also TP23.1
- net USART1_TX: now also TP5.1
- net VDD: now also S1.2 (NO_1), S1.5 (NO_2); no longer TP5.1
- net VSS: now also DR5.1
- net V_REGUSB: now also TP60.1
- net V_SWD: now also TP59.1
- net IDin: now reaches DD1.2 (A), DFet2.3 (S), DR1.2, Dfet1.3 (S), LDR.2, TP50.1
- net IDin: now also DD3.2 (A), DFet3.3 (S), DR4.2, DTVS70.1 (A1), U7.3 (SRC), U7.4 (IN)
- net at MCUC19.1, MCUR1.2, NRSTSW2.2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: now also TP65.1
- net at FB2.1, MCUR6.2, U2.59 (PB7): now also TP24.1
- net at MCUC21.1, U2.47 (VCAP_2): now also TP62.1
- net at FB1.1, MCUR5.2, U2.58 (PB6): now also TP25.1
- net at MCUC20.1, U2.31 (VCAP_1): now also TP61.1
- net at BOOTSW1.1, MCUR2.1, U2.60 (BOOT0): now also TP64.1
- new net: DTVS30.1 (A1), DTVS70.2 (A2), TP56.1
- new net: DC3.2, DR5.2, DTVS30.2 (A2), TP58.1, U7.6 (Vss), U7.7 (Pad)
- new net: DD3.1 (K), DFet3.2 (G), DR4.1, TP57.1, U7.2 (GATE)
- new net MCUCFETOFF: S1.4 (NC_2), TP66.1, U2.10 (PC2)
- new net MCUDFETOFF: S1.1 (NC_1), TP68.1, U2.9 (PC1)
- no-connect marks 36 -> 37
Other:
- note added: "Do we want to put two fets in parallel or use one to ensure we don't deal with discrepency?"
- note added: "High current ideal diode"
- note added: "Indicator LEDs - NEED to switch LEDs to correct model"
- note added: "MCU Physical E-stop"
- note added: "MCU corner"
- note removed: "Alisa's corner"
- note removed: "Indicator LEDs - Use UL current LEDS to save power ~2mA"
- moved on the sheet: BOOTSW1, FB1, FB2, FUSER2, J1, J4, J5, MCUC1, MCUC10, MCUC11, MCUC12, MCUC13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

Commit message: Library changes
Parts:
- renumbered LDR to LDR1
Changed lines of the file:
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@@
 		(dnp no)
 		(fields_autoplaced yes)
-		(property "Reference" "LDR"
+		(property "Reference" "LDR1"
 			(at 255.27 345.4399 0)
 			(show_name no)
@@
 			(project "Aqua BMS Monitor(MAIN)"
 				(path "/d7eeacc8-0d33-4ea5-a0aa-fd0653295080"
-					(reference "LDR")
+					(reference "LDR1")
 					(unit 1)
 				)

Commit message: nothing much
Parts:
- removed S1: MHPS2285N, MHPS2285N, symbol MHPS2285N:MHPS2285N
- added S1: MHPS2285N, BMS footprint lib:MHPS2285N, symbol BMS_SymbolLib:MHPS2285N
Connections:
- net CFETOFF: now also S1.3 (COM_1)
- net DFETOFF: now also S1.6 (COM_2)
- net MCUCFETOFF: now also S1.1 (NC_1)
- net MCUDFETOFF: now also S1.4 (NC_2)
- net VDD: now also S1.2 (NO_1), S1.5 (NO_2)
Changed lines of the file:
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@@
 	)
 	(symbol
-		(lib_id "MHPS2285N:MHPS2285N")
-		(at 671.83 354.33 180)
-		(unit 1)
-		(body_style 1)
-		(exclude_from_sim no)
-		(in_bom yes)
-		(on_board yes)
-		(in_pos_files yes)
-		(dnp no)
-		(property "Reference" "S1"
-			(at 662.432 361.95 0)
-			(show_name no)
-			(do_not_autoplace no)
-			(effects
-				(font
-					(size 1.27 1.27)
-				)
-				(justify left)
-			)
-		)
-		(property "Value" "MHPS2285N"
-			(at 662.432 359.41 0)
-			(show_name no)
-			(do_not_autoplace no)
-			(effects
-				(font
-					(size 1.27 1.27)
-				)
-				(justify left)
-			)
-		)
-		(property "Footprint" "MHPS2285N"
-			(at 645.16 259.41 0)
-			(hide yes)
-			(show_name no)
-			(do_not_autoplace no)
-			(effects
-				(font
-					(size 1.27 1.27)
-				)
-				(justify left top)
-			)
-		)
-		(property "Datasheet" "https://media.digikey.com/pdf/Data%20Sheets/APEM%20Components%20PDFs/MHPS_Series.pdf"
-			(at 645.16 159.41 0)
-			(hide yes)
-			(show_name no)
-			(do_not_autoplace no)
-			(effects
-				(font
-					(size 1.27 1.27)
-				)
-				(justify left top)
-			)
-		)
-		(property "Description" "Pushbutton Switches DPDT 0.1A 30V On-Mom"
-			(at 671.83 354.33 0)
-			(hide yes)
-			(show_name no)
-			(do_not_autoplace no)
-			(effects
-				(font
-					(size 1.27 1.27)
-				)
-			)
-		)
-		(property "Height" "13.5"
-			(at 645.16 -40.59 0)
-			(hide yes)
-			(show_name no)
-			(do_not_autoplace no)
-			(effects
-				(font
-					(size 1.27 1.27)
-				)
-				(justify left top)
-			)
-		)
-		(property "Mouser Part Number" "642-MHPS2285N"
-			(at 645.16 -140.59 0)
-			(hide yes)
-			(show_name no)
-			(do_not_autoplace no)
-			(effects
-				(font
-					(size 1.27 1.27)
-				)
-				(justify left top)
-			)
-		)
-		(property "Mouser Price/Stock" "https://www.mouser.co.uk/ProductDetail/Apem/MHPS2285N?qs=6hR9CYnVCPCmwxWl14NRKA%3D%3D"
-			(at 645.16 -240.59 0)
-			(hide yes)
-			(show_name no)
-			(do_not_autoplace no)
-			(effects
-				(font
-					(size 1.27 1.27)
-				)
-				(justify left top)
-			)
-		)
-		(property "Manufacturer_Name" "Apem"
-			(at 645.16 -340.59 0)
-			(hide yes)
-			(show_name no)
-			(do_not_autoplace no)
-			(effects
-				(font
-					(size 1.27 1.27)
-				)
-				(justify left top)
-			)
-		)
-		(property "Manufacturer_Part_Number" "MHPS2285N"
-			(at 645.16 -440.59 0)
-			(hide yes)
-			(show_name no)
-			(do_not_autoplace no)
-			(effects
-				(font
-					(size 1.27 1.27)
-				)
-				(justify left top)
-			)
-		)
-		(pin "1"
-		)
-		(pin "2"
-		)
-		(pin "3"
-		)
-		(pin "4"
-		)
-		(pin "5"
-		)
-		(pin "6"
-		)
-		(instances
-			(project "Aqua BMS Monitor(MAIN)"
-				(path "/d7eeacc8-0d33-4ea5-a0aa-fd0653295080"
-					(reference "S1")
-					(unit 1)
-				)
-			)
-		)
-	)
-	(symbol
 		(lib_id "Device:C")
 		(at 440.69 347.98 0)
@@
 					(unit 1)
 				)
+			)
+		)
+	)
+	(symbol
+		(lib_id "BMS_SymbolLib:MHPS2285N")
+		(at 641.35 349.25 0)
+		(unit 1)
+		(body_style 1)
+		(exclude_from_sim no)
+		(in_bom yes)
+		(on_board yes)
+		(in_pos_files yes)
+		(dnp no)
+		(fields_autoplaced yes)
+		(property "Reference" "S1"
+			(at 656.59 341.63 0)
+			(show_name no)
+			(do_not_autoplace no)
+			(effects
+				(font
+					(size 1.27 1.27)
+				)
+			)
+		)
+		(property "Value" "MHPS2285N"
+			(at 656.59 344.17 0)
+			(show_name no)
+			(do_not_autoplace no)
+			(effects
+				(font
+					(size 1.27 1.27)
+				)
+			)
+		)
+		(property "Footprint" "BMS footprint lib:MHPS2285N"
+			(at 668.02 444.17 0)
+			(hide yes)
+			(show_name no)
+			(do_not_autoplace no)
+			(effects
+				(font
+					(size 1.27 1.27)
+				)
+				(justify left top)
+			)
+		)
+		(property "Datasheet" "https://media.digikey.com/pdf/Data%20Sheets/APEM%20Components%20PDFs/MHPS_Series.pdf"
+			(at 668.02 544.17 0)
+			(hide yes)
+			(show_name no)
+			(do_not_autoplace no)
+			(effects
+				(font
+					(size 1.27 1.27)
+				)
+				(justify left top)
+			)
+		)
+		(property "Description" "Pushbutton Switches DPDT 0.1A 30V On-Mom"
+			(at 641.35 349.25 0)
+			(hide yes)
+			(show_name no)
+			(do_not_autoplace no)
+			(effects
+				(font
+					(size 1.27 1.27)
+				)
+			)
+		)
+		(property "Height" "13.5"
+			(at 668.02 744.17 0)
+			(hide yes)
+			(show_name no)
+			(do_not_autoplace no)
+			(effects
+				(font
+					(size 1.27 1.27)
+				)
+				(justify left top)
+			)
+		)
+		(property "Mouser Part Number" "642-MHPS2285N"
+			(at 668.02 844.17 0)
+			(hide yes)
+			(show_name no)
+			(do_not_autoplace no)
+			(effects
+				(font
+					(size 1.27 1.27)
+				)
+				(justify left top)
+			)
+		)
+		(property "Mouser Price/Stock" "https://www.mouser.co.uk/ProductDetail/Apem/MHPS2285N?qs=6hR9CYnVCPCmwxWl14NRKA%3D%3D"
+			(at 668.02 944.17 0)
+			(hide yes)
+			(show_name no)
+			(do_not_autoplace no)
+			(effects
+				(font
+					(size 1.27 1.27)
+				)
+				(justify left top)
+			)
+		)
+		(property "Manufacturer_Name" "Apem"
+			(at 668.02 1044.17 0)
+			(hide yes)
+			(show_name no)
+			(do_not_autoplace no)
+			(effects
+				(font
+					(size 1.27 1.27)
+				)
+				(justify left top)
+			)
+		)
+		(property "Manufacturer_Part_Number" "MHPS2285N"
+			(at 668.02 1144.17 0)
+			(hide yes)
+			(show_name no)
+			(do_not_autoplace no)
+			(effects
+				(font
+					(size 1.27 1.27)
+				)
+				(justify left top)
+			)
+		)
+		(pin "4"
+		)
+		(pin "6"
+		)
+		(pin "2"
+		)
+		(pin "5"
+		)
+		(pin "1"
+		)
+		(pin "3"
+		)
+		(instances
+			(project "Aqua BMS Monitor(MAIN)"
+				(path "/d7eeacc8-0d33-4ea5-a0aa-fd0653295080"
+					(reference "S1")
+					(unit 1)
+				)
