File: Aqua BMS Monitor(MAIN).kicad_sch (KiCad schematic)
At the start: 249 parts, among them J1 UART Jpins, J4 USB_C_Receptacle_USB2.0_14P, J5 SWD_01x04_Pin, Q13 NMOS, Q6 NPN, U1 BQ7695202, U2 STM32F205RETx, U3 AMS1117-3.3, U4 LM66100DCKR, U5 LM66100DCKR, U6 LM66100DCKR, U7 LTC4359-DCB, X1 X322516MRB4SI

Commit message: Maybe a mess, maybe a good thing
Parts:
- U1: footprint easyeda2kicad:BQ7695202PFBR -> BMS footprint lib:QFP50P900X900X120-48N
Changed lines of the file:
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@@
 			)
 		)
-		(property "Footprint" "easyeda2kicad:BQ7695202PFBR"
+		(property "Footprint" "BMS footprint lib:QFP50P900X900X120-48N"
 			(at 436.88 193.548 0)
 			(hide yes)

Commit message: Final changes, pushing merging with main
Parts:
- TP1: value BAT+TP -> BATplusTP; footprint (none) -> TestPoint:TestPoint_Pad_D1.5mm
- TP10, TP11, TP12, TP13, TP14, TP15, TP16, TP17, TP18, TP19, TP20, TP21, TP22, TP23, TP24, TP25, TP26, TP27, TP28, TP29, TP30, TP31, TP32, TP33, TP34, TP35, TP36, TP37, TP38, TP39, TP40, TP41, TP42, TP43, TP44, TP45, TP46, TP47, TP48, TP49, TP5, TP50, TP51, TP52, TP53, TP54, TP55, TP56, TP57, TP58, TP59, TP6, TP60, TP61, TP62, TP63, TP64, TP65, TP66, TP67, TP68, TP69, TP70, TP71, TP72, TP8: footprint (none) -> TestPoint:TestPoint_Pad_D1.5mm
- TP7: footprint (none) -> TestPoint:TestPoint_Pad_1.5x1.5mm
- TP9: value PWR+TP -> PWRplusTP; footprint (none) -> TestPoint:TestPoint_Pad_D1.5mm

Commit message: Please work
Parts:
- removed J4: USB_C_Receptacle_USB2.0_14P, symbol Connector:USB_C_Receptacle_USB2.0_14P
- removed U3: AMS1117-3.3, Package_TO_SOT_SMD:SOT-223-3_TabPin2, symbol Regulator_Linear:AMS1117-3.3
- added U8: GT-USB-7035C, easyeda2kicad:14P_USB-C_Female, symbol easyeda2kicad symbols:GT-USB-7035C
- added U9: AMS1117-3.3, Package_TO_SOT_SMD:SOT-223-3_TabPin2, symbol Regulator_Linear:AMS1117-3.3
- BR1, XRC5, Xshun1: footprint easyeda2kicad:100_R1210 -> easyeda2kicad:100_3W_R2512
- CR1, CR2, CR3, CR4, CR5: footprint easyeda2kicad:50_R0603 -> easyeda2kicad:50_100mW_R0805
- DTVS30: footprint (none) -> easyeda2kicad:30V_TVS_Diode
- DTVS70: footprint (none) -> easyeda2kicad:70V_TVS_Diode
- LED1, LED2, LED3, LED4, LED5: footprint (none) -> easyeda2kicad:LED0805-RD
- Q6: footprint easyeda2kicad:NPN_BJT -> easyeda2kicad:100_330mW_R1210
- RR1: footprint easyeda2kicad:300_R0805 -> easyeda2kicad:300_250mW_R1206
- SC1, SC2, SC3, XC1, XC2, XC3, XC4, XC5, XCshun1: footprint Capacitor_SMD:C_1210_3225Metric_Pad1.33x2.70mm_HandSolder -> easyeda2kicad:0.1uF_C1210
- SRinN1, SRinP1: footprint easyeda2kicad:100_R1210 -> easyeda2kicad:100_330mW_R1210
- U1: footprint BMS footprint lib:QFP50P900X900X120-48N -> easyeda2kicad:BQ7695202PFBR
- XCreg1: footprint Capacitor_SMD:C_1210_3225Metric_Pad1.33x2.70mm_HandSolder -> easyeda2kicad:0.47 uF_C1210
- XRreg1: footprint easyeda2kicad:5_RES-SMD_L6.4-W3.8 -> easyeda2kicad:5_1W_R2512
Connections:
- net USB_D+: now also USBR3.2, U8.A6 (D+), U8.B6 (D+); no longer USBR3.1
- net USB_D-: now also U8.A7 (D-), U8.B7 (D-)
- net VDD: now also USBR3.1; no longer USBR3.2
- net VSS: now also USBR2.1, U8.1 (GND), U8.2 (GND), U8.3 (GND), U8.4 (GND), U8.A1 (GND), U8.A12 (GND), U8.B1 (GND), U8.B12 (GND), U9.1 (GND); no longer USBR2.2
- net V_REGUSB: now also U9.2 (VO)
- net USB_C_VBUS: now reaches USBC1.1
- net USB_C_VBUS: now also U8.A4 (VBUS), U8.A9 (VBUS), U8.B4 (VBUS), U8.B9 (VBUS), U9.3 (VI)
- net at USBR1.1: now also U8.A5 (CC1)
- new net: U8.B5 (CC2), USBR2.2
- no-connect marks 37 -> 36
Other:
- note removed: "1.8k typical value in datasheet?"
- note removed: "PA9"
- moved on the sheet: BOOTSW1, FB1, FB2, MCUC19, MCUC20, MCUC21, MCUR1, MCUR2, MCUR3, MCUR4, MCUR5, MCUR6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

Commit message: Added Male XT60s
Parts:
- removed MainBattIn1: Main lines, symbol Connector:Conn_01x02_Pin
- added U10, U11, U12, U3: XT60, easyeda2kicad:XT60_M, symbol easyeda2kicad symbols:XT60
Connections:
- net BAT+: now also U3.2 (+)
- net CPACK+: now also U11.2 (+)
- net DPACK+: now also U12.2 (+)
- net PACK-: now also U11.1 (-), U12.1 (-)
- net PWR+: now also U10.2 (+)
- net VSS: now also U10.1 (-), U3.1 (-)
Other:
- moved on the sheet: TP7

Commit message: Cleaned up netlist and schematic
Parts:
- removed 3TFuse1: (no value), symbol Device:3TerminalFuse
- removed Cellin1: 1 low 5 high, symbol Connector:Conn_01x05_Pin
- removed ChFet1, DFet2, DFet3, Dfet1, FFet1, Q13: NMOS, easyeda2kicad:NMOS, symbol Simulation_SPICE:NMOS
- added 3TFuse1: SCF9550-45-07, easyeda2kicad:FUSE-SMD_3P-L9.5-W5.0_SFK-5030X, symbol easyeda2kicad symbols:SCF9550-45-07
- added Cellin1: 1 low 5 high, easyeda2kicad:CONN-TH_B5B-XH-A-LF-SN, symbol easyeda2kicad symbols:B5B-XH-A
- added ChFet1, DFet2, DFet3, Dfet1, FFet1, NMOS1: NMOS, easyeda2kicad:NMOS, symbol easyeda2kicad symbols:H7534N
- J5: footprint M20_8890445:HARWIN_M20-8890445 -> easyeda2kicad:HARWIN_M20-8890445
- Q6: footprint easyeda2kicad:100_330mW_R1210 -> easyeda2kicad:NPN_BJT
- S1: footprint BMS footprint lib:MHPS2285N -> easyeda2kicad:MHPS2285N
- U10, U11, U12, U3: footprint easyeda2kicad:XT60_M -> easyeda2kicad:CONN-TH_XT60
Connections:
- net BAT+: now also 3TFuse1.1
- net CD: now also 3TFuse1.2, ChFet1.5 (D), DFet2.5 (D), Dfet1.5 (D)
- net DPACK+: now also DFet3.1 (S), DFet3.2 (S), DFet3.3 (S), NMOS1.5 (D)
- net FUSE: now also FFet1.4 (G)
- net IDin: now also DFet2.1 (S), DFet2.2 (S), DFet2.3 (S), DFet3.5 (D), Dfet1.1 (S), Dfet1.2 (S), Dfet1.3 (S)
- net V1: now also Cellin1.2
- net V2: now also Cellin1.3
- net V3: now also Cellin1.4
- net V4: now also Cellin1.5
- net VSS: now also Cellin1.1, FFet1.5 (D)
- net at DRgate1.2: now also Dfet1.4 (G)
- net at DD3.1 (K), DR4.1, TP57.1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: now also DFet3.4 (G)
- net at ChD2.1 (K), ChR1.1, ChR2.2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: now also ChFet1.4 (G)
- net at DD1.1 (K), DD2.1 (K), DR1.1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: now also NMOS1.1 (S), NMOS1.2 (S), NMOS1.3 (S)
- net at D17.1 (K), R46.1, R47.2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: now also NMOS1.4 (G)
- net at ChD1.1 (K): now also ChFet1.1 (S), ChFet1.2 (S), ChFet1.3 (S)
- net at DRgate2.2: now also DFet2.4 (G)
- new net: 3TFuse1.3, FFet1.1 (S), FFet1.2 (S), FFet1.3 (S)
Other:
- note removed: "Why? Reduce power loss through Rds? Yes"

Commit message: Updates
- PCB organisation
- Some reroutes on schematic
- Adding new components for fake bat/cells
Parts:
- removed D4: 100V, easyeda2kicad:100V_Schottky, symbol Device:D_Schottky
- added PWRtoBAT1, SWShunt5: SW_Push, easyeda2kicad:SW_Push_YZA-009, symbol Switch:SW_Push
Connections:
- net BAT+: now also PWRtoBAT1.1
- net DPACK+: now also DFet3.5 (D), NMOS1.1 (S), NMOS1.2 (S), NMOS1.3 (S); no longer DFet3.1 (S), DFet3.2 (S), DFet3.3 (S), NMOS1.5 (D)
- net IDin: now also DFet3.1 (S), DFet3.2 (S), DFet3.3 (S); no longer DFet3.5 (D)
- net PWR+: now also PWRtoBAT1.2
- net VSS: now also FFet1.1 (S), FFet1.2 (S), FFet1.3 (S), SWShunt5.2; no longer FFet1.5 (D), Rshunt1.2
- net at DD1.1 (K), DD2.1 (K), DR1.1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: now also NMOS1.5 (D); no longer NMOS1.1 (S), NMOS1.2 (S), NMOS1.3 (S)
- new net: 3TFuse1.3, FFet1.5 (D)
- new net: Rshunt1.2, SWShunt5.1
Other:
- note added: "PBat - voltage divider"
- note added: "PSeudoCell - voltage divider"
- note removed: "PSeudoCell - voltage divider - F"
- moved on the sheet: DFet3, FFet1

Commit message: PCB and schem arrangement/changes
Connections:
- net CD: now also ChFet1.1 (S), ChFet1.2 (S), ChFet1.3 (S); no longer ChFet1.5 (D)
- net DSG: now also DD2.1 (K)
- net at DD1.1 (K), DR1.1, DR2.2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: no longer DD2.1 (K)
- new net: ChD1.1 (K), ChFet1.5 (D)
Other:
- moved on the sheet: ChFet1, DD2, DR2

Commit message: Renamed a folder to fix routing issue in library
Parts:
- removed U10, U11, U12, U3: XT60, easyeda2kicad:CONN-TH_XT60, symbol easyeda2kicad symbols:XT60
- added DFet4: NMOS, easyeda2kicad:NMOS, symbol easyeda2kicad symbols:H7534N
- added DFetGate3, DFetGate4: 10, Resistor_SMD:R_0805_2012Metric, symbol BQ76952PFBR:R
- added J2, J3, J4, J6: XT60PW-M, BMS footprint lib:AMASS_XT60PW-M, symbol Xt-60PW-M:XT60PW-M
- C1-0, C2-0, CC2-1, CC3-2, CC4-3: footprint easyeda2kicad:220nF_C1210 -> Capacitor_SMD:C_0603_1608Metric
- SC1, SC2, SC3, XC1, XC2, XC3, XC4, XC5, XCshun1: footprint easyeda2kicad:0.1uF_C1210 -> Capacitor_SMD:C_0603_1608Metric
Connections:
- net BAT+: now also J2.1 (P)
- net CPACK+: now also J6.1 (P)
- net DPACK+: now also DFet4.4 (G), DFet4.5 (D), DFetGate4.2, J4.1 (P)
- net IDin: now also DFet4.1 (S), DFet4.2 (S), DFet4.3 (S)
- net PACK-: now also J4.2 (N), J6.2 (N)
- net PWR+: now also J3.1 (P)
- net VSS: now also J2.2 (N), J3.2 (N)
- net at DD3.1 (K), DR4.1, TP57.1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: now also DFetGate3.1, DFetGate4.1; no longer DFet3.4 (G)
- new net: J3.SH1 (SHIELD), J3.SH2 (SHIELD)
- new net: J4.SH1 (SHIELD), J4.SH2 (SHIELD)
- new net: J2.SH1 (SHIELD), J2.SH2 (SHIELD)
- new net: J6.SH1 (SHIELD), J6.SH2 (SHIELD)
- new net: DFet3.4 (G), DFetGate3.2
- no-connect marks 36 -> 40
Other:
- note removed: "Needs NET tie to ground, I think this is not right..."
- moved on the sheet: DC3, DD3, DFet3, DR4, DR5, DTVS30, DTVS70, TP1, TP56, TP57, TP58, TP9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
