File: Aqua BMS Monitor(MAIN).kicad_sch (KiCad schematic)
At the start: 256 parts, among them J1 UART Jpins, J2 XT60PW-M, J3 XT60PW-M, J4 XT60PW-M, J5 SWD_01x04_Pin, J6 XT60PW-M, J7 USB_C_Female_USB2_Small, Q6 NPN, U1 BQ7695202, U2 STM32F205RETx, U4 LM66100DCKR, U5 LM66100DCKR, U6 LM66100DCKR, U7 LTC4359-DCB, U9 AMS1117-3.3, X1 X322516MRB4SI

Commit message: Grinding on the power line :)
Parts:
- removed DTVS30: D_TVS_Filled, easyeda2kicad:30V_TVS_Diode, symbol Device:D_TVS_Filled
- removed DTVS70: D_TVS_Filled, easyeda2kicad:70V_TVS_Diode, symbol Device:D_TVS_Filled
- removed LED4: XZCM2CRK53WA-8VF, easyeda2kicad:LED0805-RD, symbol Device:LED
- removed LEDR4: 1k, easyeda2kicad:1k_R1206, symbol BQ76952PFBR:R
- removed PWRtoBAT1, SWShunt1, SWShunt2, SWShunt3, SWShunt4, SWShunt5: SW_Push, easyeda2kicad:SW_Push_YZA-009, symbol Switch:SW_Push
- added D1: SMF7V0A, Diode_SMD:D_SMF, symbol Diode:SMF7V0A
- added D2: SMF30A, Diode_SMD:D_SMF, symbol Diode:SMF30A
- added S2, S3, S4, S5, S6: EG1218, BMS footprint lib:SW_EG1218, symbol EG1218:EG1218
- added better1: (no value), BMS footprint lib:1101A2CQEA-Switch, symbol BMS_SymbolLib:Trying_1101A2CQEA
- ChC1, ChC2, DC1, DC2, FC1, PCc2, PcC1, PdC1, PdC2: footprint easyeda2kicad:0.1uF_C1210 -> Capacitor_SMD:C_0603_1608Metric
- ChR1, DR1, DR4, PcR2, PdR2, R46: footprint easyeda2kicad:10M_R1210 -> Resistor_SMD:R_0603_1608Metric
- DFetGate3, DFetGate4: footprint Resistor_SMD:R_0805_2012Metric -> Resistor_SMD:R_0603_1608Metric
- FR1: footprint easyeda2kicad:20k_R1206 -> Resistor_SMD:R_0603_1608Metric
- LDR1, R47: footprint easyeda2kicad:10k_R1206 -> Resistor_SMD:R_0603_1608Metric
- PdR1: footprint easyeda2kicad:1k_R1206 -> Resistor_SMD:R_0603_1608Metric
- TP22: value DpackTP -> ChGpackTP; footprint TestPoint:TestPoint_Pad_D1.5mm -> TestPoint:TestPoint_Pad_D1.0mm
- TP27, TP44, TP48, TP51, TP56, TP57, TP58: footprint TestPoint:TestPoint_Pad_D1.5mm -> TestPoint:TestPoint_Pad_D1.0mm
Connections:
- net BAT: no longer LEDR5.2
- net BAT+: now also better1.2 (Comm), better1.3 (Off)
- net DPACK+: no longer DFet4.4 (G), DFetGate4.2
- net IDin: now also D1.1 (A1)
- net PWR+: now also LEDR5.2, S2.3, better1.1 (On)
- net V1: now also S5.1, S5.2
- net V2: now also S4.1, S4.2
- net V3: now also S3.1, S3.2
- net V4: now also S2.1, S2.2
- net VSS: now also S6.1, S6.2
- net at TP56.1: now also D1.2 (A2), D2.2 (A2)
- net at DC3.2, DR5.2, TP58.1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: now also D2.1 (A1)
- net at Rshunt2.1, Rshunt3.2: now also S4.3
- net at Rshunt1.1, Rshunt2.2: now also S5.3
- net at Rshunt3.1, Rshunt4.2: now also S3.3
- net at Rshunt1.2: now also S6.3
- new net: DFet4.4 (G), DFetGate4.2
Other:
- moved on the sheet: DFetGate4

Commit message: All done routing the main power lines
Parts:
- removed TP19: REG18TP, TestPoint:TestPoint_Pad_D1.5mm, symbol Connector:TestPoint
- removed TP45: Reg2TP, TestPoint:TestPoint_Pad_D1.5mm, symbol Connector:TestPoint
- removed TP47: ReginTP, TestPoint:TestPoint_Pad_D1.5mm, symbol Connector:TestPoint
- removed TP56: IDTVSTP, TestPoint:TestPoint_Pad_D1.0mm, symbol Connector:TestPoint
- DR2: footprint easyeda2kicad:1k_R1206 -> Resistor_SMD:R_0603_1608Metric
- RC2: footprint easyeda2kicad:22nF_C1210 -> Capacitor_SMD:C_0402_1005Metric
- RR2: footprint easyeda2kicad:10M_R1210 -> Resistor_SMD:R_0603_1608Metric
- TP13, TP14, TP46, TP49, TP53, TP54, TP55: footprint TestPoint:TestPoint_Pad_D1.5mm -> TestPoint:TestPoint_Pad_D1.0mm
Connections:
- net CACK+ is gone; now on net CPACK+: LEDR3.2
- net PACK-: now also LED2.1 (K), LED3.1 (K)
- net VSS: no longer LED2.1 (K), LED3.1 (K)

Commit message: Just a freaking mess
Connections:
- net SCL: now also TP25.1; no longer MCUTVS1.2
- net SDA: now also TP24.1; no longer MCUTVS2.2
- net at FB2.1, MCUR6.2, U2.59 (PB7): now also MCUTVS2.2; no longer TP24.1
- net at FB1.1, MCUR5.2, U2.58 (PB6): now also MCUTVS1.2; no longer TP25.1
Other:
- moved on the sheet: MCUTVS1, MCUTVS2, TP24, TP25

Commit message: Just disturbing to look at tbh
Parts:
- removed MCUC1, MCUC10, MCUC2, MCUC3, MCUC4, MCUC5, MCUC6, MCUC7, MCUC8, MCUC9: 100 nF, easyeda2kicad:100nF_C0402, symbol Device:C
Other:
- moved on the sheet: MCUC11, MCUC12, MCUC13, MCUC14, MCUC15, MCUC16

Commit message: Plsplsplsplspls
Parts:
- added TP19: VSSTP, TestPoint:TestPoint_Pad_1.5x1.5mm, symbol Connector:TestPoint
- added TsC1, TsC2: 470 pF, easyeda2kicad:470pF_C0402, symbol Device:C
- TsC3: renamed from TsC1; footprint easyeda2kicad:470pF_C0805 -> easyeda2kicad:470pF_C0402
- TsR1: footprint easyeda2kicad:10k_R1206 -> easyeda2kicad:10k_62.5mW_R0402
Connections:
- net TS1: now also TsC1.1
- net TS3: now also TsC2.1
- net VSS: now also TP19.1, TsC1.2, TsC2.2
Other:
- moved on the sheet: TH2, TP15, TP17, TsR1, TsRST1A

Commit message: minor changes
Parts:
- removed TP19: VSSTP, TestPoint:TestPoint_Pad_1.5x1.5mm, symbol Connector:TestPoint
- TP53: value ClampGateTP -> CmpG
Changed lines of the file:
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@@
 	)
 	(junction
-		(at 144.78 187.96)
-		(diameter 0)
-		(color 0 0 0 0)
-	)
-	(junction
 		(at 222.25 326.39)
 		(diameter 0)
@@
 	(wire
 		(pts
-			(xy 144.78 187.96) (xy 144.78 190.5)
+			(xy 144.78 184.15) (xy 144.78 190.5)
 		)
 		(stroke
@@
 	(wire
 		(pts
-			(xy 144.78 184.15) (xy 144.78 187.96)
-		)
-		(stroke
-			(width 0)
-			(type default)
-		)
-	)
-	(wire
-		(pts
 			(xy 220.98 360.68) (xy 220.98 364.49)
 		)
@@
 	)
 	(symbol
-		(lib_id "Connector:TestPoint")
-		(at 144.78 187.96 270)
-		(unit 1)
-		(body_style 1)
-		(exclude_from_sim no)
-		(in_bom yes)
-		(on_board yes)
-		(in_pos_files yes)
-		(dnp no)
-		(fields_autoplaced yes)
-		(property "Reference" "TP19"
-			(at 149.86 186.6899 90)
-			(show_name no)
-			(do_not_autoplace no)
-			(effects
-				(font
-					(size 1.27 1.27)
-				)
-				(justify left)
-			)
-		)
-		(property "Value" "VSSTP"
-			(at 149.86 189.2299 90)
-			(show_name no)
-			(do_not_autoplace no)
-			(effects
-				(font
-					(size 1.27 1.27)
-				)
-				(justify left)
-			)
-		)
-		(property "Footprint" "TestPoint:TestPoint_Pad_1.5x1.5mm"
-			(at 144.78 193.04 0)
-			(hide yes)
-			(show_name no)
-			(do_not_autoplace no)
-			(effects
-				(font
-					(size 1.27 1.27)
-				)
-			)
-		)
-		(property "Datasheet" ""
-			(at 144.78 193.04 0)
-			(hide yes)
-			(show_name no)
-			(do_not_autoplace no)
-			(effects
-				(font
-					(size 1.27 1.27)
-				)
-			)
-		)
-		(property "Description" "test point"
-			(at 144.78 187.96 0)
-			(hide yes)
-			(show_name no)
-			(do_not_autoplace no)
-			(effects
-				(font
-					(size 1.27 1.27)
-				)
-			)
-		)
-		(pin "1"
-		)
-		(instances
-			(project "Aqua BMS Monitor(MAIN)"
-				(path "/d7eeacc8-0d33-4ea5-a0aa-fd0653295080"
-					(reference "TP19")
-					(unit 1)
-				)
-			)
-		)
-	)
-	(symbol
 		(lib_id "power:VSS")
 		(at 25.4 109.22 180)
@@
 			)
 		)
-		(property "Value" "ClampGateTP"
+		(property "Value" "CmpG"
 			(at 283.718 347.472 90)
 			(show_name no)

Commit message: Not sure
Parts:
- added MCUTVS3, MCUTVS4: PTVSUC3D5VB, easyeda2kicad:5V_TVS_SOD-323_L1.8-W1.3-LS2.5-BI, symbol 5V_TVS_BI:PTVSUC3D5VB
Connections:
- net USART1_RX: now also MCUTVS4.2
- net USART1_TX: now also MCUTVS3.2
- net VSS: now also MCUTVS3.1, MCUTVS4.1
Other:
- moved on the sheet: J1, S1, TP23, TP5, TP66, TP67, TP68, TP69
