File: Aqua BMS Monitor(MAIN).kicad_pcb (KiCad board)
At the start: 2 copper layers, 259 parts, among them J1 UART Jpins, J5 SWD_01x04_Pin, Q13 NMOS, Q6 NPN, U1 BQ7695202, U10 XT60, U11 XT60, U12 XT60, U2 STM32F205RETx, U3 XT60, U4 LM66100DCKR, U5 LM66100DCKR, U6 LM66100DCKR, U7 LTC4359-DCB, U8 GT-USB-7035C, U9 AMS1117-3.3, X1 X322516MRB4SI

Commit message: Updates
- PCB organisation
- Some reroutes on schematic
- Adding new components for fake bat/cells
Parts:
- removed the 3TFuse1 at (184.9, 76.1)
- removed D4: 100V, easyeda2kicad:100V_Schottky
- removed the FFet1 at (183.1, 107.1)
- removed Q13: NMOS, easyeda2kicad:NMOS
- added PWRtoBAT1: SW_Push, easyeda2kicad:SW_Push_YZA-009, F.Cu at (-140.0, 229.0)
- added SWShunt5: SW_Push, easyeda2kicad:SW_Push_YZA-009, F.Cu at (-129.0, 229.0)
- moved Rshunt4 346.6 mm to (-140.7, 218.5)
- moved SWShunt4 332.6 mm to (-129.4, 219.8)
- moved SWShunt3 329.7 mm to (-128.6, 210.5)
- moved SWShunt2 327.7 mm to (-129.2, 200.2)
- moved Rshunt3 326.7 mm to (-141.2, 210.5)
- moved SWShunt1 325.3 mm to (-129.2, 190.0)
- moved Rshunt2 324.5 mm to (-141.0, 201.0)
- moved Rshunt1 322.6 mm to (-140.5, 193.0)
- moved Cellin1 276.2 mm to (-80.9, 188.8)
- moved XRC5 266.7 mm to (-56.9, 185.8)
- moved MCUR1 252.7 mm to (408.0, 40.8)
- moved DTVS70 252.4 mm to (-19.6, -23.0)
- moved U4 250.5 mm to (396.6, 29.8)
- moved U6 250.5 mm to (403.0, 29.8)
- moved U5 250.5 mm to (399.8, 29.8)
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Connections:
- 3TFuse1 pad 3: Net-(3TFuse1-Pad3) -> Net-(FFet1-D)
- DFet3 pad 1: DPACK+ -> IDin
- DFet3 pad 2: DPACK+ -> IDin
- DFet3 pad 3: DPACK+ -> IDin
- DFet3 pad 5: IDin -> DPACK+
- FFet1 pad 1: Net-(3TFuse1-Pad3) -> BAT-
- FFet1 pad 2: Net-(3TFuse1-Pad3) -> BAT-
- FFet1 pad 3: Net-(3TFuse1-Pad3) -> BAT-
- FFet1 pad 5: BAT- -> Net-(FFet1-D)
- NMOS1 pad 1: Net-(DD1-K) -> DPACK+
- NMOS1 pad 2: Net-(DD1-K) -> DPACK+
- NMOS1 pad 3: Net-(DD1-K) -> DPACK+
- NMOS1 pad 5: DPACK+ -> Net-(DD1-K)
- Rshunt1 pad 2: BAT- -> Net-(Rshunt1-Pad2)
Other:
- board text added: "BAT circuit"
- board text added: "Cell management"
- board text added: "Charge"
- board text added: "Clamp"
- board text added: "Discharge Charge"
- board text added: "Fake cells Setup"
- board text added: "Fuse Setup"
- board text added: "IDeal diode"
- board text added: "LEDs"
- board text added: "MCU"
- board text added: "Regulator circuit"
- board text added: "Shunt resistor setup"
- board text added: "TPs"
- board text added: "Thermal measurement"

Commit message: Update Aqua BMS Monitor(MAIN).kicad_pcb
Parts:
- moved PWRtoBAT1 267.1 mm to (66.0, 59.0), turned to -90 degrees
- moved Cellin1 187.8 mm to (54.0, 58.1), turned to -90 degrees
- moved Rshunt3 175.4 mm to (-20.3, 83.5)
- moved SWShunt1 174.9 mm to (-8.85, 63.0)
- moved SWShunt2 174.9 mm to (-8.85, 73.2)
- moved SWShunt3 174.9 mm to (-8.31, 83.5)
- moved SWShunt4 174.9 mm to (-9.06, 92.8)
- moved Rshunt1 174.9 mm to (-20.2, 66.0)
- moved Rshunt2 174.9 mm to (-20.7, 74.0)
- moved Rshunt4 174.9 mm to (-20.4, 91.5)
- moved SWShunt5 174.9 mm to (-8.74, 102.0)
- moved BQ296115DSGR1 157.7 mm to (78.5, 135.8)
- moved C1-0 157.7 mm to (54.0, 115.5)
- moved C2-0 157.7 mm to (54.5, 124.8)
- moved CC2-1 157.7 mm to (55.5, 134.2)
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
Commit message: PCB and schem arrangement/changes
Parts:
- removed the ChFet1 at (-51.0, 85.3)
- removed the DFet2 at (-54.0, 39.3)
- removed the Dfet1 at (-55.0, 48.3)
- moved DC1 225.4 mm to (151.0, 71.5), turned to -90 degrees
- moved PcC1 221.0 mm to (130.5, 31.0)
- moved ChC2 220.5 mm to (143.5, 52.0)
- moved PcR2 219.6 mm to (136.0, 35.6), turned to 90 degrees
- moved DC2 218.9 mm to (151.5, 76.0)
- moved PdC2 217.0 mm to (108.5, 129.0)
- moved PCc2 215.3 mm to (135.5, 31.0)
- moved ChC1 214.6 mm to (143.5, 47.5), turned to -90 degrees
- moved PcR3 204.0 mm to (127.6, 40.0)
- moved PdC1 201.6 mm to (97.0, 129.0)
- moved ChD2 201.0 mm to (117.0, 50.0), turned to 90 degrees
- moved PackR1 200.7 mm to (136.5, 48.5), turned to 90 degrees
- moved DD1 199.7 mm to (121.5, 62.5), turned to -90 degrees
- moved DR2 198.1 mm to (120.5, 57.0), turned to 180 degrees
- moved PcFet1 195.1 mm to (130.0, 35.4), turned to 180 degrees
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Connections:
- ChFet1 pad 1: Net-(ChD1-K) -> CD
- ChFet1 pad 2: Net-(ChD1-K) -> CD
- ChFet1 pad 3: Net-(ChD1-K) -> CD
- ChFet1 pad 5: CD -> Net-(ChD1-K)
- DD2 pad 1: Net-(DD1-K) -> DSG
Other:
- board text added: "Pre-Discharge Charge"
- board text removed: "Discharge Charge"

Commit message: Renamed a folder to fix routing issue in library
Parts:
- removed U10, U11, U12, U3: XT60, easyeda2kicad:CONN-TH_XT60
- added DFet4: NMOS, easyeda2kicad:NMOS, F.Cu at (-4.32, -14.9)
- added DFetGate3: 10, Resistor_SMD:R_0805_2012Metric, F.Cu at (-9.29, -16.5)
- added DFetGate4: 10, Resistor_SMD:R_0805_2012Metric, F.Cu at (-9.29, -13.6)
- added J2: XT60PW-M, BMS footprint lib:AMASS_XT60PW-M, F.Cu at (141.9, -11.9)
- added J3: XT60PW-M, BMS footprint lib:AMASS_XT60PW-M, F.Cu at (160.8, -11.9)
- added J4: XT60PW-M, BMS footprint lib:AMASS_XT60PW-M, F.Cu at (179.6, -11.9)
- added J6: XT60PW-M, BMS footprint lib:AMASS_XT60PW-M, F.Cu at (198.5, -11.9)
- C1-0, C2-0, CC2-1, CC3-2, CC4-3: footprint easyeda2kicad:220nF_C1210 -> Capacitor_SMD:C_0603_1608Metric
- SC1, SC2, SC3, XC1, XC2, XC3, XC4, XC5, XCshun1: footprint easyeda2kicad:0.1uF_C1210 -> Capacitor_SMD:C_0603_1608Metric
- moved SC2 4.27 mm to (281.0, 78.5)
Connections:
- DFet3 pad 4: Net-(DD3-K) -> Net-(DFet3-G)

Commit message: more changes
Parts:
- BMSC1: footprint easyeda2kicad:220nF_C1210 -> Capacitor_SMD:C_0603_1608Metric
- moved BQ296115DSGR1 166.7 mm to (44.0, 89.8)
- moved C1-0 166.7 mm to (19.5, 69.5)
- moved C2-0 166.7 mm to (20.0, 78.8)
- moved CC2-1 166.7 mm to (21.0, 88.2)
- moved CC3-2 166.7 mm to (22.5, 97.0)
- moved CC4-3 166.7 mm to (22.3, 104.0)
- moved CR1 166.7 mm to (90.2, 107.5)
- moved CR2 166.7 mm to (92.0, 96.8)
- moved CR3 166.7 mm to (79.5, 88.2)
- moved CR4 166.7 mm to (74.2, 88.2)
- moved CR5 166.7 mm to (83.0, 88.8)
- moved XC1 166.7 mm to (61.0, 85.0)
- moved XC2 166.7 mm to (60.0, 93.5)
- moved XC3 166.7 mm to (39.8, 68.0)
- moved XC4 166.7 mm to (38.5, 79.0)
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Other:
- board text added: "BAT in circuit"
- board text added: "Charge and discharge"
- board text removed: "Charge"

Commit message: More changes - lots of uncertainty
Parts:
- BMSC1, C1-0, C2-0, CC2-1, CC3-2, CC4-3, SC1, SC2, SC3, XC1, XC2, XC3, XC4, XC5: footprint Capacitor_SMD:C_0603_1608Metric -> Capacitor_SMD:C_0402_1005Metric
- SRinN1, SRinP1: footprint easyeda2kicad:100_330mW_R1210 -> Resistor_SMD:R_0402_1005Metric
- moved TP8 266.6 mm to (140.0, 95.0)
- moved C4 148.2 mm to (136.6, 94.5)
- moved SRinN1 140.6 mm to (136.0, 96.5), turned to -90 degrees
- moved SRinP1 138.5 mm to (137.0, 96.5), turned to -90 degrees
- moved FRShunt1 131.8 mm to (136.2, 112.0)
- moved SC3 131.3 mm to (136.5, 93.0)
- moved C1-0 116.5 mm to (134.0, 91.0)
- moved CC4-3 112.5 mm to (132.0, 79.0), turned to 90 degrees
- moved C2-0 112.3 mm to (131.5, 92.0), turned to 180 degrees
- moved CC2-1 110.1 mm to (131.1, 91.0), turned to 180 degrees
- moved CC3-2 109.3 mm to (131.5, 89.0), turned to 180 degrees
- moved BQ296115DSGR1 83.8 mm to (116.2, 132.1), turned to -90 degrees
- moved Cellin1 71.7 mm to (115.0, 97.9)
- moved PWRtoBAT1 70.5 mm to (-39.5, 192.0)
- moved BC1 70.5 mm to (-19.5, 205.9)
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