File: Aqua BMS Monitor(MAIN).kicad_pcb (KiCad board)
At the start: 4 copper layers, 142 x 93 mm, 250 parts, among them J1 UART Jpins, J2 XT60PW-M, J3 XT60PW-M, J4 XT60PW-M, J5 SWD_01x04_Pin, J6 XT60PW-M, J7 USB_C_Female_USB2_Small, Q6 NPN, U1 BQ7695202, U2 STM32F205RETx, U4 LM66100DCKR, U5 LM66100DCKR, U6 LM66100DCKR, U7 LTC4359-DCB, U9 AMS1117-3.3, X1 X322516MRB4SI

Commit message: Just a freaking mess
Parts:
- moved MCUR5 263.7 mm to (161.5, 84.5)
- moved MCUR6 261.5 mm to (161.5, 86.9), turned to 90 degrees
- moved OSCC1 253.8 mm to (161.6, 93.5), turned to -90 degrees
- moved OSCC2 253.8 mm to (161.5, 96.5)
- moved X1 253.5 mm to (159.5, 94.5)
- moved MCUC19 252.7 mm to (164.0, 95.5), turned to 180 degrees
- moved U5 252.4 mm to (166.0, 81.0)
- moved U9 252.4 mm to (172.0, 80.5)
- moved USBC1 252.4 mm to (177.5, 78.0)
- moved USBC2 252.4 mm to (177.5, 82.5)
- moved C71 252.4 mm to (166.1, 78.5)
- moved BOOTSW1 251.7 mm to (192.4, 75.5)
- moved C70 251.7 mm to (182.9, 84.0)
- moved J1 251.7 mm to (193.4, 103.0)
- moved J7 251.7 mm to (190.9, 94.0)
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Connections:
- MCUTVS1 pad 2: SCL -> Net-(U2-PB6)
- MCUTVS2 pad 2: SDA -> Net-(U2-PB7)
- TP24 pad 1: Net-(U2-PB7) -> SDA
- TP25 pad 1: Net-(U2-PB6) -> SCL
Routing:
- net ALERT: track 2.00 -> 41.7 mm, vias 0 -> 2
- net Net-(U2-NRST): track 42.2 -> 12.4 mm
- net SDA: track 0.00 -> 20.9 mm
- net Net-(U2-BOOT0): track 30.6 -> 11.8 mm
- net SCL: track 0.00 -> 17.1 mm
- net Net-(U2-PB6): track 2.52 -> 18.6 mm
- net SWDIO: track 19.2 -> 4.32 mm
- net Net-(U2-PB7): track 2.00 -> 16.0 mm
- net SWCLK: track 19.5 -> 6.96 mm
- net USB_C_VBUS: track 25.9 -> 14.9 mm
- net OSC_IN: track 7.22 -> 10.1 mm
- net OSC_OUT: track 5.30 -> 7.79 mm

Commit message: We getting there
Parts:
- moved S1 238.0 mm to (158.5, 99.5), turned to 0 degrees
- moved C72 219.8 mm to (172.0, 91.0)
- moved U6 219.8 mm to (172.5, 89.0)
- moved TP5 182.3 mm to (190.0, 99.0)
- moved TP23 177.3 mm to (197.5, 105.0)
- moved TP62 158.3 mm to (188.5, 90.5)
- moved TP61 155.6 mm to (189.0, 105.0)
- moved MCUR1 43.3 mm to (174.5, 91.5), turned to 180 degrees
- moved MCUR2 38.5 mm to (178.5, 89.0), turned to 180 degrees
- moved OSCC2 10.0 mm to (171.5, 96.5)
- moved X1 10.0 mm to (169.5, 94.5)
- moved OSCC1 9.96 mm to (171.5, 93.0)
- moved MCUC17 9.60 mm to (174.0, 99.5)
- moved MCUC18 9.60 mm to (173.0, 99.5)
- moved MCUC19 9.50 mm to (173.5, 95.5)
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Routing:
- net DCHG: track 0.00 -> 55.8 mm, vias 0 -> 2
- net DDSG: track 0.00 -> 47.0 mm, vias 0 -> 2
- net RST_SHUT: track 0.05 -> 45.6 mm, vias 0 -> 2
- net CFETOFF: track 0.00 -> 30.7 mm, vias 0 -> 1
- net Net-(U2-NRST): track 12.4 -> 41.8 mm
- net VDD: track 39.8 -> 68.8 mm
- net DFETOFF: track 0.00 -> 24.7 mm, vias 0 -> 1
- net MCUDFETOFF: track 0.00 -> 23.6 mm, vias 0 -> 1
- net MCUCFETOFF: track 0.00 -> 20.2 mm, vias 0 -> 1
- net Net-(U2-BOOT0): track 11.8 -> 29.6 mm
- net BAT-: track 185.8 -> 202.8 mm, vias 57 -> 59
- net SWDIO: track 4.32 -> 19.2 mm
- net USB_C_VBUS: track 14.9 -> 29.3 mm
- net SWCLK: track 6.96 -> 19.5 mm
- net ALERT: track 41.7 -> 52.4 mm
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Other:
- board size 142 x 93 mm -> 142 x 101.5 mm

Commit message: Just disturbing to look at tbh
Parts:
- removed MCUC1, MCUC10, MCUC2, MCUC3, MCUC4, MCUC5, MCUC6, MCUC7, MCUC8, MCUC9: 100 nF, easyeda2kicad:100nF_C0402
- moved TP64 179.1 mm to (198.8, 81.5)
- moved TP65 179.1 mm to (197.5, 75.0)
- moved TP59 164.9 mm to (187.0, 108.2)
- moved TP60 149.2 mm to (175.5, 74.2)
- moved TP24 146.9 mm to (166.5, 88.5)
- moved TP25 142.1 mm to (163.8, 83.8)
- moved TP68 139.3 mm to (173.8, 105.5)
- moved TP66 138.3 mm to (168.8, 98.2)
- moved TP63 136.3 mm to (170.0, 105.5)
- moved TP67 129.3 mm to (157.8, 88.8)
- moved TP70 122.9 mm to (162.2, 105.5)
- moved TP69 120.2 mm to (151.8, 89.2)
- moved TP72 104.1 mm to (153.2, 83.0)
- moved TP71 102.8 mm to (147.2, 89.0)
- moved C70 23.0 mm to (191.5, 107.0)
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Routing:
- net VDD: track 68.8 -> 166.3 mm, vias 0 -> 7
- net Net-(U2-BOOT0): track 29.6 -> 53.5 mm, vias 2 -> 4
- net REG1: track 8.56 -> 27.7 mm, vias 0 -> 2
- net BAT-: track 202.8 -> 214.9 mm, vias 59 -> 82
- net USART1_TX: track 19.5 -> 30.0 mm, vias 0 -> 3
- net MCUDFETOFF: track 23.6 -> 28.7 mm
- net SWCLK: track 19.5 -> 23.7 mm
- net Net-(U2-PB6): track 18.5 -> 22.2 mm
- net Net-(U2-NRST): track 41.8 -> 45.4 mm, vias 3 -> 5
- net RST_SHUT: track 45.6 -> 49.1 mm, vias 2 -> 3
- net DDSG: track 47.0 -> 50.2 mm, vias 2 -> 3
- net V_SWD: track 6.34 -> 9.36 mm
- net DCHG: track 55.8 -> 58.4 mm, vias 2 -> 3
- net Net-(U2-VCAP_1): track 7.90 -> 5.44 mm
- net V_REGUSB: track 7.53 -> 9.78 mm
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
Commit message: Plsplsplsplspls
Parts:
- added TP19: VSSTP, TestPoint:TestPoint_Pad_1.5x1.5mm, F.Cu at (148.5, 91.8)
- added TsC1: 470 pF, easyeda2kicad:470pF_C0402, F.Cu at (139.5, 93.0)
- added TsC2: 470 pF, easyeda2kicad:470pF_C0402, F.Cu at (144.5, 93.5)
- TsC3: renamed from TsC1; footprint easyeda2kicad:470pF_C0805 -> easyeda2kicad:470pF_C0402
- TsR1: footprint easyeda2kicad:10k_R1206 -> easyeda2kicad:10k_62.5mW_R0402
- moved TH1 153.4 mm to (139.8, 94.0)
- moved TsRST1 152.5 mm to (145.0, 96.0)
- moved TP12 143.0 mm to (141.5, 96.5)
- moved TP17 141.3 mm to (141.5, 99.0)
- moved TsR1 131.7 mm to (148.5, 96.4), turned to -90 degrees
- moved TH3 128.7 mm to (147.0, 58.0)
- moved TP15 126.8 mm to (144.5, 91.5)
- moved TsC3 122.2 mm to (147.0, 59.5)
- moved TP18 114.8 mm to (143.5, 58.5)
- moved TH2 15.9 mm to (266.5, 39.5)
- moved TP6 1.27 mm to (134.0, 97.5)
- moved TP8 1.26 mm to (139.0, 97.5)
- moved BMSC1 0.69 mm to (140.5, 88.5)
- moved Dfet1 0.53 mm to (147.2, 55.0)
- moved DFet2 0.53 mm to (147.3, 62.5)
Routing:
- net HDQ: track 0.00 -> 42.3 mm, vias 0 -> 3
- net TS2: track 0.00 -> 13.5 mm
- net BAT-: track 214.9 -> 222.5 mm, vias 82 -> 89
- net Net-(U1-REG18): track 1.01 -> 8.29 mm
- net TS1: track 4.01 -> 10.5 mm, vias 0 -> 1
- net TS3: track 0.00 -> 2.23 mm
- net Net-(TsRST1A-B): track 0.00 -> 1.46 mm
- net SRN: track 11.6 -> 12.5 mm

Commit message: minor changes
Parts:
- removed TP19: VSSTP, TestPoint:TestPoint_Pad_1.5x1.5mm
- TP53: value ClampGateTP -> CmpG
- moved TP72 3.51 mm to (156.8, 82.8)
Routing:
- net RST_SHUT: track 49.1 -> 52.0 mm
- net BAT-: track 222.5 -> 221.8 mm

Commit message: Small fixes
Parts:
- moved TP25 3.34 mm to (160.5, 84.5)
- moved TP24 3.20 mm to (164.0, 86.5)
- moved C72 2.92 mm to (163.5, 90.5), turned to 90 degrees
- moved TP7 2.69 mm to (127.5, 99.0)
- moved TP15 2.50 mm to (142.0, 91.5)
- moved TP17 2.00 mm to (143.5, 99.0)
- moved U6 1.58 mm to (161.5, 90.0), turned to 90 degrees
- moved TP68 1.25 mm to (175.0, 105.5)
- moved TP71 1.25 mm to (146.0, 89.0)
- moved TsC2 1.12 mm to (143.5, 93.0)
- moved TP70 0.50 mm to (162.2, 105.0)
- turned TsR1 to 90 degrees
Routing:
- net REG1: track 27.7 -> 34.5 mm
- net Net-(U1-REG18): track 8.29 -> 2.39 mm
- net TS3: track 2.23 -> 7.45 mm
- net BAT-: track 221.8 -> 218.0 mm, vias 89 -> 90
- net SWCLK: track 23.7 -> 20.7 mm
- net VDD: track 166.3 -> 168.9 mm, vias 7 -> 6
- net RST_SHUT: track 52.0 -> 54.5 mm
- net DDSG: track 50.2 -> 48.8 mm
- net Net-(U2-BOOT0): track 53.5 -> 55.0 mm
- net CFETOFF: track 32.3 -> 33.4 mm
- net SCL: track 28.3 -> 27.3 mm
- net DCHG: track 58.1 -> 59.0 mm
- net SDA: track 31.3 -> 30.7 mm
- net SWDIO: track 19.6 -> 20.2 mm
- net USB_C_VBUS: track 31.3 -> 30.8 mm

Commit message: Minors
Parts:
- moved U6 6.75 mm to (168.2, 90.0), turned to -90 degrees
- moved C72 2.93 mm to (166.2, 89.5), turned to -90 degrees
- moved TP24 2.02 mm to (164.2, 88.5)
- moved TP12 0.56 mm to (141.0, 96.2)
- moved MCUC14 0.41 mm to (188.8, 92.2), turned to -90 degrees
- moved MCUC19 0.30 mm to (173.3, 95.8)
- moved BMSC1 0.27 mm to (140.5, 88.8)
- moved TP15 0.25 mm to (142.0, 91.2)
Routing:
- net BAT-: track 218.0 -> 205.0 mm, vias 90 -> 92
- net DPACK+: track 5.57 -> 14.8 mm
- net VDD: track 168.9 -> 164.5 mm
- net BAT+: track 49.0 -> 51.7 mm
- net Net-(BQ296115DSGR1-V3): track 7.37 -> 9.41 mm
- net Net-(BQ296115DSGR1-V4): track 9.38 -> 11.4 mm
- net REG1: track 34.5 -> 33.0 mm
- net Net-(Dfet1-G): track 19.9 -> 21.0 mm
- net Net-(U1-REG18): track 2.39 -> 1.52 mm
- net TS1: track 10.7 -> 10.1 mm
- net Net-(U2-BOOT0): track 55.0 -> 55.5 mm
- net Net-(DFet2-G): track 16.7 -> 16.2 mm
- net V_SWD: track 9.36 -> 9.87 mm
- net USART1_TX: vias 3 -> 2
- net USART1_RX: vias 3 -> 2
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
Commit message: Revamping
Parts:
- moved TP25 44.8 mm to (177.5, 126.0)
- moved TP61 44.7 mm to (155.0, 131.0)
- moved TP24 43.7 mm to (185.0, 127.0)
- moved TP72 43.3 mm to (157.5, 126.0)
- moved NRSTSW2 40.7 mm to (191.3, 115.0)
- moved TP67 39.5 mm to (171.0, 126.0)
- moved TP69 39.1 mm to (165.0, 126.0)
- moved TP71 37.8 mm to (150.5, 126.5)
- moved BOOTSW1 35.8 mm to (198.3, 115.0), turned to 180 degrees
- moved TP70 34.7 mm to (189.5, 126.5)
- moved TP66 34.3 mm to (162.5, 132.0)
- moved TP68 26.5 mm to (174.0, 132.0)
- moved TP63 26.1 mm to (168.0, 131.5)
- moved TP5 18.5 mm to (208.0, 94.0)
- moved MCUR1 17.0 mm to (168.3, 104.5), turned to 90 degrees
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Routing:
- net DCHG: track 59.0 -> 4.77 mm, vias 3 -> 1
- net RST_SHUT: track 54.5 -> 3.80 mm, vias 3 -> 1
- net DDSG: track 48.8 -> 2.49 mm, vias 3 -> 0
- net ALERT: track 53.4 -> 9.13 mm, vias 4 -> 1
- net CFETOFF: track 33.4 -> 0.00 mm, vias 2 -> 0
- net DFETOFF: track 26.4 -> 1.71 mm, vias 2 -> 1
- net HDQ: track 42.6 -> 19.1 mm, vias 2 -> 1
- net REG1: track 33.0 -> 10.7 mm, vias 2 -> 0
- net MCUCFETOFF: track 21.7 -> 0.00 mm, vias 2 -> 0
- net MCUDFETOFF: track 28.9 -> 8.14 mm
- net BAT-: track 205.0 -> 221.2 mm, vias 92 -> 91
- net Net-(DD1-K): track 41.7 -> 32.5 mm
- net Net-(U2-NRST): track 45.5 -> 37.0 mm, vias 5 -> 2
- net Net-(U2-BOOT0): track 55.5 -> 47.4 mm, vias 4 -> 2
- net VDD: track 164.5 -> 170.7 mm
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